File: PTP_Teo_Sencar_Project1.kicad_pcb (KiCad board)
At the start: 2 copper layers, 45 parts, among them J1 Screw_Terminal_01x02, SW1 SW_Push, SW2 SW_SPDT_312, U1 LM2574N-5, U2 4027, U3 4027, U4 74LS47, U5 FYS-3911BUHR-21, U6 74LVC1G11, U7 NE555P

Commit message: Spajanje vodova
Parts:
- moved R16 3.50 mm to (177.0, 96.5)
- moved R14 3.00 mm to (177.0, 93.0)
Routing:
- net +5V: track 0.00 -> 212.9 mm, vias 0 -> 4
- net Q1: track 0.00 -> 62.5 mm, vias 0 -> 3
- net Q0: track 0.00 -> 60.5 mm, vias 0 -> 4
- net Q3: track 0.00 -> 54.4 mm, vias 0 -> 2
- net Net-(D4-K): track 0.00 -> 51.5 mm, vias 0 -> 2
- net 555: track 0.00 -> 48.8 mm, vias 0 -> 2
- net Clock: track 0.00 -> 45.0 mm, vias 0 -> 2
- net Net-(U4-a): track 0.00 -> 42.9 mm
- net Reset: track 0.00 -> 40.4 mm, vias 0 -> 2
- net Net-(U4-b): track 0.00 -> 39.7 mm
- net Net-(U4-c): track 0.00 -> 38.1 mm
- net Net-(U3A-J): track 0.00 -> 33.4 mm, vias 0 -> 2
- net Q2: track 0.00 -> 32.3 mm, vias 0 -> 2
- net Net-(SW2-A): track 0.00 -> 27.7 mm, vias 0 -> 2
- net Net-(U2B-J): track 0.00 -> 27.3 mm, vias 0 -> 2
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- added copper zone on B.Cu, net GND

Commit message: Gerber fileovi, BOM
Routing:
- net GND: track 1.26 -> 43.3 mm, vias 0 -> 4
- net Net-(U2A-J): track 17.7 -> 25.5 mm, vias 2 -> 4
- net Net-(U5-B): track 19.6 -> 16.7 mm
- net 555: track 48.8 -> 50.9 mm
- net Net-(U4-d): track 10.5 -> 11.9 mm
- net Net-(U5-C): track 9.94 -> 11.2 mm
- net Net-(U4-e): track 14.6 -> 15.2 mm
- net Net-(U7-DIS): track 23.6 -> 24.1 mm
- net Q1: track 62.5 -> 62.1 mm, vias 3 -> 4
Other:
- board outline added: 100 x 80 mm
- board text added: "PTP - BCD counter Teo Senčar"
